File: Hardware/PCB/auto_irrigator.kicad_sch (KiCad schematic)
At the start: 51 parts, among them J1 GND 12V, J10 FLOW3, J2 VALVE1, J3 VALVE2, J4 VALVE3, J5 VALVE4, J6 I2C1, J7 FLOW4, J8 FLOW1, J9 FLOW2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

Commit message: AutoIrrigator rev 2
Aggiunte notifiche. Migliorata ulteriormente la stabilità. Modificata PCB per sistemare gli errori della rev 1.
Parts:
- removed P1: ~, power_symbols:stm_headers, symbol power_symbols:stm_headers
- added C7: 100nF, Capacitor_SMD:C_0603_1608Metric, symbol Device:C
- added J11: ~, headers:swdio, symbol headers:swdio
- added J12: FLOW5, Connector_JST:JST_EH_B3B-EH-A_1x03_P2.50mm_Vertical, symbol Connector_Generic:Conn_01x03
- added Q9: AO3400A, Package_TO_SOT_SMD:SOT-23, symbol Transistor_FET:AO3400A
- added R13: 10K, Resistor_SMD:R_0603_1608Metric, symbol Device:R
- added R14: 5K1, Resistor_SMD:R_0603_1608Metric, symbol Device:R
- added R15: 1K8, Resistor_SMD:R_0603_1608Metric, symbol Device:R
Connections:
- net +12V: now also J12.3 (Pin_3), R14.2
- net +3V3: now also J11.1 (3V3)
- net GND: now also C7.2, J11.2 (GND), J12.1 (Pin_1), Q9.2 (S), R13.2, R15.1
- net SWCLK: now also J11.3 (SWCLK)
- net SWDIO: now also J11.4 (SWDIO)
- net BAT_ADC: now reaches U1.12 (PA5)
- net BAT_ADC: now also C7.1, R14.1, R15.2
- net SCL renamed FLOW5
- net FLOW5: now also Q9.3 (D)
- new net: J12.2 (Pin_2), Q9.1 (G), R13.1
- no-connect marks 4 -> 2
Other:
- moved on the sheet: J10, J7, J8, J9, Q5, Q6, Q7, Q8, R11, R12, R7, R8
